File: BQ34Z100EVM.kicad_sch (KiCad schematic)
At the start: 46 parts, among them IC1 BQ34Z100PWR-G1, IC2 SN74HC164PWR, J1 Conn_01x05_Pin, J2 Screw_Terminal_01x04, Q3 2N7002, Q4 2N7002, Q5 BSS84, SW1 SW_Push

Commit message: minor changes
Parts:
- J2: footprint TerminalBlock_MetzConnect:TerminalBlock_MetzConnect_Type055_RT01504HDWU_1x04_P5.00mm_Horizontal -> TerminalBlock_Phoenix:TerminalBlock_Phoenix_MKDS-1,5-4-5.08_1x04_P5.08mm_Horizontal
Connections:
- net at R30.1, R6.1: now also J2.3 (Pin_3); no longer J2.1 (Pin_1)
- net at Q3.3 (D), Q5.2 (S), R2.1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: now also J2.1 (Pin_1); no longer J2.3 (Pin_3)
Other:
- note added: "B+"
- note added: "B-"
- note added: "Pack-"
- moved on the sheet: J2
Changed lines of the file:
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@@
 	(generator_version "9.0")
 	(paper "A4")
+	(text "B+"
+		(exclude_from_sim no)
+		(at 32.004 123.444 0)
+		(effects
+			(font
+				(size 1.27 1.27)
+			)
+		)
+	)
+	(text "B-"
+		(exclude_from_sim no)
+		(at 32.004 125.984 0)
+		(effects
+			(font
+				(size 1.27 1.27)
+			)
+		)
+	)
+	(text "Pack-"
+		(exclude_from_sim no)
+		(at 32.004 128.27 0)
+		(effects
+			(font
+				(size 1.27 1.27)
+			)
+		)
+	)
 	(junction
 		(at 101.6 58.42)
@@
 	)
 	(junction
+		(at 62.23 128.27)
+		(diameter 0)
+		(color 0 0 0 0)
+	)
+	(junction
 		(at 255.27 60.96)
 		(diameter 0)
@@
 	(junction
 		(at 95.25 118.11)
-		(diameter 0)
-		(color 0 0 0 0)
-	)
-	(junction
-		(at 62.23 128.27)
 		(diameter 0)
 		(color 0 0 0 0)
@@
 	)
 	(no_connect
-		(at 41.91 120.65)
+		(at 41.91 130.81)
 	)
 	(no_connect
@@
 	(wire
 		(pts
-			(xy 54.61 125.73) (xy 41.91 125.73)
-		)
-		(stroke
-			(width 0)
-			(type default)
-		)
-	)
-	(wire
-		(pts
-			(xy 62.23 128.27) (xy 41.91 128.27)
-		)
-		(stroke
-			(width 0)
-			(type default)
-		)
-	)
-	(wire
-		(pts
 			(xy 264.16 85.09) (xy 264.16 87.63)
 		)
@@
 	(wire
 		(pts
+			(xy 41.91 128.27) (xy 62.23 128.27)
+		)
+		(stroke
+			(width 0)
+			(type default)
+		)
+	)
+	(wire
+		(pts
 			(xy 240.03 60.96) (xy 240.03 69.85)
 		)
@@
 	(wire
 		(pts
+			(xy 41.91 123.19) (xy 50.8 123.19)
+		)
+		(stroke
+			(width 0)
+			(type default)
+		)
+	)
+	(wire
+		(pts
 			(xy 81.28 128.27) (xy 95.25 128.27)
 		)
@@
 	(wire
 		(pts
-			(xy 41.91 123.19) (xy 50.8 123.19)
-		)
-		(stroke
-			(width 0)
-			(type default)
-		)
-	)
-	(wire
-		(pts
 			(xy 59.69 168.91) (xy 66.04 168.91)
 		)
@@
 		(pts
 			(xy 71.12 78.74) (xy 66.04 78.74)
+		)
+		(stroke
+			(width 0)
+			(type default)
+		)
+	)
+	(wire
+		(pts
+			(xy 41.91 125.73) (xy 54.61 125.73)
 		)
 		(stroke
@@
 	(symbol
 		(lib_id "Connector:Screw_Terminal_01x04")
-		(at 36.83 125.73 180)
+		(at 36.83 125.73 0)
+		(mirror y)
 		(unit 1)
 		(exclude_from_sim no)
@@
 		(on_board yes)
 		(dnp no)
-		(fields_autoplaced yes)
 		(property "Reference" "J2"
-			(at 36.83 114.3 0)
+			(at 36.83 137.16 0)
 			(effects
 				(font
@@
 		)
 		(property "Value" "Screw_Terminal_01x04"
-			(at 36.83 116.84 0)
+			(at 36.83 134.62 0)
 			(effects
 				(font
@@
 			)
 		)
-		(property "Footprint" "TerminalBlock_MetzConnect:TerminalBlock_MetzConnect_Type055_RT01504HDWU_1x04_P5.00mm_Horizontal"
+		(property "Footprint" "TerminalBlock_Phoenix:TerminalBlock_Phoenix_MKDS-1,5-4-5.08_1x04_P5.08mm_Horizontal"
 			(at 36.83 125.73 0)
 			(effects
