File: BQ34Z100EVM.kicad_pcb (KiCad board)
At the start: 2 copper layers, 110.5 x 34 mm, 46 parts, among them IC1 BQ34Z100PWR-G1, IC2 SN74HC164PWR, J1 Conn_01x05_Pin, J2 Screw_Terminal_01x04, Q3 2N7002, Q4 2N7002, Q5 BSS84, SW1 SW_Push

Commit message: added minor changes
Parts:
- D1, D2, D3, D4, D5: footprint Resistor_SMD:R_1206_3216Metric_Pad1.30x1.75mm_HandSolder -> LED_SMD:LED_1206_3216Metric_Pad1.42x1.75mm_HandSolder
- J2: footprint TerminalBlock_MetzConnect:TerminalBlock_MetzConnect_Type055_RT01504HDWU_1x04_P5.00mm_Horizontal -> TerminalBlock_Phoenix:TerminalBlock_Phoenix_MKDS-1,5-4-5.08_1x04_P5.08mm_Horizontal
- R30: footprint Resistor_SMD:R_1206_3216Metric_Pad1.30x1.75mm_HandSolder -> Resistor_SMD:R_2512_6332Metric_Pad1.40x3.35mm_HandSolder
- moved J2 14.9 mm to (75.7, 100.1), turned to -90 degrees
- moved J1 2.51 mm to (173.1, 102.9)
- moved C6 0.16 mm to (91.9, 120.6)
Connections:
- Q3 pad 3: Net-(J2-Pin_3) -> Net-(J2-Pin_1)
- Q5 pad 2: Net-(J2-Pin_3) -> Net-(J2-Pin_1)
- R2 pad 1: Net-(J2-Pin_3) -> Net-(J2-Pin_1)
- R3 pad 1: Net-(J2-Pin_3) -> Net-(J2-Pin_1)
- R30 pad 1: Net-(J2-Pin_1) -> Net-(J2-Pin_3)
- R6 pad 1: Net-(J2-Pin_1) -> Net-(J2-Pin_3)
Routing:
- net /SRN: track 0.00 -> 60.2 mm, vias 0 -> 2
- net /SRP: track 0.00 -> 58.0 mm, vias 0 -> 2
- net Net-(IC1-VEN): track 0.00 -> 53.8 mm, vias 0 -> 2
- net Net-(IC1-BAT): track 0.00 -> 49.6 mm, vias 0 -> 3
- net Net-(J2-Pin_1): track 0.00 -> 41.5 mm
- net /REGIN: track 73.5 -> 111.0 mm
- net Net-(Q5-G): track 0.00 -> 22.7 mm, vias 0 -> 4
- net /P2: track 0.00 -> 22.3 mm, vias 0 -> 2
- net Net-(J2-Pin_3): track 0.00 -> 16.9 mm
- net Net-(J2-Pin_2): track 0.00 -> 16.5 mm
- net Net-(IC2-QE): track 0.00 -> 16.5 mm, vias 0 -> 2
- net Net-(Q5-D): track 0.00 -> 15.5 mm
- net Net-(Q3-G): track 0.00 -> 9.22 mm
- net Net-(Q4-D): track 0.00 -> 7.12 mm
- net Net-(J1-Pin_1): track 20.5 -> 25.2 mm
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- added copper zone on B.Cu, net GND
- added copper zone on F.Cu, net GND
Other:
- outline, holes or cut-outs redrawn
- board text added: "B+"
- board text added: "B-"
- board text added: "BQ34Z100 EVB"
- board text added: "GND"
- board text added: "HDQ"
- board text added: "P-"
- board text added: "SCL"
- board text added: "SDA"
- board text added: "VCC"

Commit message: minor changes
Changed lines of the file:
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@@
 		(tags "Zener Diode")
 		(property "Reference" "Z2"
-			(at 0 -2.9 90)
+			(at 0 2.8 90)
 			(layer "F.SilkS")
 			(effects
